File: circuit/Make_3.3V.sch (KiCad schematic (older format))
At the start: 3 parts, among them U3 033EZ1H

Commit message: Servoのchを4->6に変更
Parts:
- renumbered C3 to C2, C4 to C3
Changed lines of the file:
@@
 LIBS:contrib
 LIBS:valves
+LIBS:stm32
 LIBS:robocon_sch
+LIBS:SamacSys_Parts
 LIBS:YASU
-LIBS:stm32
 LIBS:ServoDriver-cache
 EELAYER 25 0
@@
 $Descr A4 11693 8268
 encoding utf-8
-Sheet 2 6
+Sheet 6 6
 Title ""
 Date ""
@@
 $EndComp
 $Comp
-L GND #PWR026
+L GND #PWR062
 U 1 1 58DB517B
 P 6550 3250
-F 0 "#PWR026" H 6550 3000 50  0001 C CNN
+F 0 "#PWR062" H 6550 3000 50  0001 C CNN
 F 1 "GND" H 6550 3100 50  0000 C CNN
 F 2 "" H 6550 3250 50  0000 C CNN
@@
 $EndComp
 $Comp
-L +3.3V #PWR027
+L +3.3V #PWR063
 U 1 1 58DB51E7
 P 5400 2850
-F 0 "#PWR027" H 5400 2700 50  0001 C CNN
+F 0 "#PWR063" H 5400 2700 50  0001 C CNN
 F 1 "+3.3V" H 5400 2990 50  0000 C CNN
 F 2 "" H 5400 2850 50  0000 C CNN
@@
 Connection ~ 5850 3050
 $Comp
-L C C3
+L C C2
 U 1 1 58DB5268
 P 5850 3300
-F 0 "C3" H 5875 3400 50  0000 L CNN
+F 0 "C2" H 5875 3400 50  0000 L CNN
 F 1 "0.1u" H 5875 3200 50  0000 L CNN
 F 2 "Capacitors_SMD:C_0805_HandSoldering" H 5888 3150 50  0001 C CNN
@@
 $EndComp
 $Comp
-L C C4
+L C C3
 U 1 1 58DB5295
 P 6250 3300
-F 0 "C4" H 6275 3400 50  0000 L CNN
+F 0 "C3" H 6275 3400 50  0000 L CNN
 F 1 "47u" H 6275 3200 50  0000 L CNN
 F 2 "Capacitors_SMD:C_1210_HandSoldering" H 6288 3150 50  0001 C CNN

Commit message: チップ抵抗の大きさ変更とガーバー出力のための手直し
Parts:
- C2: footprint Capacitors_SMD:C_0805_HandSoldering -> Capacitors_SMD:C_0603_HandSoldering
Changed lines of the file:
@@
 F 0 "C2" H 5875 3400 50  0000 L CNN
 F 1 "0.1u" H 5875 3200 50  0000 L CNN
-F 2 "Capacitors_SMD:C_0805_HandSoldering" H 5888 3150 50  0001 C CNN
+F 2 "Capacitors_SMD:C_0603_HandSoldering" H 5888 3150 50  0001 C CNN
 F 3 "" H 5850 3300 50  0000 C CNN
 	1    5850 3300
