File: circuit/RotarySW.sch (KiCad schematic (older format))
At the start: 5 parts, among them SW1 SW_ROTARY

Commit message: Servoのchを4->6に変更
Parts:
- renumbered R4 to R6, R5 to R7, R6 to R8, R7 to R9
Changed lines of the file:
@@
 LIBS:contrib
 LIBS:valves
+LIBS:stm32
 LIBS:robocon_sch
+LIBS:SamacSys_Parts
 LIBS:YASU
-LIBS:stm32
 LIBS:ServoDriver-cache
 EELAYER 25 0
@@
 $Descr A4 11693 8268
 encoding utf-8
-Sheet 3 6
+Sheet 4 6
 Title ""
 Date ""
@@
 $EndComp
 $Comp
-L +3.3V #PWR034
+L +3.3V #PWR030
 U 1 1 5936F694
 P 5650 2250
-F 0 "#PWR034" H 5650 2100 50  0001 C CNN
+F 0 "#PWR030" H 5650 2100 50  0001 C CNN
 F 1 "+3.3V" H 5650 2390 50  0000 C CNN
 F 2 "" H 5650 2250 50  0000 C CNN
@@
 $EndComp
 $Comp
-L GND #PWR035
+L GND #PWR031
 U 1 1 5936F69A
 P 5650 3250
-F 0 "#PWR035" H 5650 3000 50  0001 C CNN
+F 0 "#PWR031" H 5650 3000 50  0001 C CNN
 F 1 "GND" H 5650 3100 50  0000 C CNN
 F 2 "" H 5650 3250 50  0000 C CNN
@@
 $EndComp
 $Comp
-L R R7
+L R R9
 U 1 1 5936F6A0
 P 5650 2550
-F 0 "R7" V 5730 2550 50  0000 C CNN
+F 0 "R9" V 5730 2550 50  0000 C CNN
 F 1 "10k" V 5650 2550 50  0000 C CNN
 F 2 "Resistors_SMD:R_0603_HandSoldering" V 5580 2550 50  0001 C CNN
@@
 $EndComp
 $Comp
-L R R6
+L R R8
 U 1 1 5936F6A7
 P 5500 2550
-F 0 "R6" V 5580 2550 50  0000 C CNN
+F 0 "R8" V 5580 2550 50  0000 C CNN
 F 1 "10k" V 5500 2550 50  0000 C CNN
 F 2 "Resistors_SMD:R_0603_HandSoldering" V 5430 2550 50  0001 C CNN
@@
 $EndComp
 $Comp
-L R R5
+L R R7
 U 1 1 5936F6AE
 P 5350 2550
-F 0 "R5" V 5430 2550 50  0000 C CNN
+F 0 "R7" V 5430 2550 50  0000 C CNN
 F 1 "10k" V 5350 2550 50  0000 C CNN
 F 2 "Resistors_SMD:R_0603_HandSoldering" V 5280 2550 50  0001 C CNN
@@
 $EndComp
 $Comp
-L R R4
+L R R6
 U 1 1 5936F6B5
 P 5200 2550
-F 0 "R4" V 5280 2550 50  0000 C CNN
+F 0 "R6" V 5280 2550 50  0000 C CNN
 F 1 "10k" V 5200 2550 50  0000 C CNN
 F 2 "Resistors_SMD:R_0603_HandSoldering" V 5130 2550 50  0001 C CNN

Commit message: ロータリースイッチの配線終わり
Parts:
- R9: footprint Resistors_SMD:R_0603_HandSoldering -> Resistors_THT:R_Axial_DIN0207_L6.3mm_D2.5mm_P7.62mm_Horizontal
Changed lines of the file:
@@
 F 0 "R9" V 5730 2550 50  0000 C CNN
 F 1 "10k" V 5650 2550 50  0000 C CNN
-F 2 "Resistors_SMD:R_0603_HandSoldering" V 5580 2550 50  0001 C CNN
+F 2 "Resistors_THT:R_Axial_DIN0207_L6.3mm_D2.5mm_P7.62mm_Horizontal" V 5580 2550 50  0001 C CNN
 F 3 "" H 5650 2550 50  0000 C CNN
 	1    5650 2550

Commit message: チップ抵抗の大きさ変更とガーバー出力のための手直し
Parts:
- R6, R7, R8: footprint Resistors_SMD:R_0603_HandSoldering -> YASU:R_0603_HandSoldering_LP
Changed lines of the file:
@@
 F 0 "R8" V 5580 2550 50  0000 C CNN
 F 1 "10k" V 5500 2550 50  0000 C CNN
-F 2 "Resistors_SMD:R_0603_HandSoldering" V 5430 2550 50  0001 C CNN
+F 2 "YASU:R_0603_HandSoldering_LP" V 5430 2550 50  0001 C CNN
 F 3 "" H 5500 2550 50  0000 C CNN
 	1    5500 2550
@@
 F 0 "R7" V 5430 2550 50  0000 C CNN
 F 1 "10k" V 5350 2550 50  0000 C CNN
-F 2 "Resistors_SMD:R_0603_HandSoldering" V 5280 2550 50  0001 C CNN
+F 2 "YASU:R_0603_HandSoldering_LP" V 5280 2550 50  0001 C CNN
 F 3 "" H 5350 2550 50  0000 C CNN
 	1    5350 2550
@@
 F 0 "R6" V 5280 2550 50  0000 C CNN
 F 1 "10k" V 5200 2550 50  0000 C CNN
-F 2 "Resistors_SMD:R_0603_HandSoldering" V 5130 2550 50  0001 C CNN
+F 2 "YASU:R_0603_HandSoldering_LP" V 5130 2550 50  0001 C CNN
 F 3 "" H 5200 2550 50  0000 C CNN
 	1    5200 2550
