File: circuit/ServoDriver.sch (KiCad schematic (older format))
At the start: 9 parts, among them U1 STM32F042K6Tx

Commit message: 基板加工用にデータを変更したやつを追加
Parts:
- BT1: footprint YASU:XT_M -> YASU:XT_Mdot
Changed lines of the file:
@@
 F 0 "BT1" H 10700 1800 50  0000 L CNN
 F 1 "Battery_Cell" H 10700 1700 50  0000 L CNN
-F 2 "YASU:XT_M" V 10600 1760 50  0001 C CNN
+F 2 "YASU:XT_Mdot" V 10600 1760 50  0001 C CNN
 F 3 "" V 10600 1760 50  0001 C CNN
 	1    10600 1700

Commit message: チップ抵抗の大きさ変更とガーバー出力のための手直し
Parts:
- C1: footprint Capacitors_SMD:C_0805_HandSoldering -> Capacitors_SMD:C_0603_HandSoldering
- R1, R2, R3: footprint Resistors_SMD:R_0603_HandSoldering -> YASU:R_0603_HandSoldering_LP
Changed lines of the file:
@@
 F 0 "C1" H 5375 2950 50  0000 L CNN
 F 1 "0.1u" H 5375 2750 50  0000 L CNN
-F 2 "Capacitors_SMD:C_0805_HandSoldering" H 5388 2700 50  0001 C CNN
+F 2 "Capacitors_SMD:C_0603_HandSoldering" H 5388 2700 50  0001 C CNN
 F 3 "" H 5350 2850 50  0001 C CNN
 	1    5350 2850
@@
 F 0 "R3" V 10180 2050 50  0000 C CNN
 F 1 "1k" V 10100 2050 50  0000 C CNN
-F 2 "Resistors_SMD:R_0603_HandSoldering" V 10030 2050 50  0001 C CNN
+F 2 "YASU:R_0603_HandSoldering_LP" V 10030 2050 50  0001 C CNN
 F 3 "" H 10100 2050 50  0001 C CNN
 	1    10100 2050
@@
 F 0 "R1" V 1780 5850 50  0000 C CNN
 F 1 "1k" V 1700 5850 50  0000 C CNN
-F 2 "Resistors_SMD:R_0603_HandSoldering" V 1630 5850 50  0001 C CNN
+F 2 "YASU:R_0603_HandSoldering_LP" V 1630 5850 50  0001 C CNN
 F 3 "" H 1700 5850 50  0001 C CNN
 	1    1700 5850
@@
 F 0 "R2" V 8430 5500 50  0000 C CNN
 F 1 "1k" V 8350 5500 50  0000 C CNN
-F 2 "Resistors_SMD:R_0603_HandSoldering" V 8280 5500 50  0001 C CNN
+F 2 "YASU:R_0603_HandSoldering_LP" V 8280 5500 50  0001 C CNN
 F 3 "" H 8350 5500 50  0001 C CNN
 	1    8350 5500
